File: BreadBatt.kicad_pcb (KiCad board)
At the start: 2 copper layers, 58.4 x 20.3 mm, 27 parts, among them J1 +5Vin, J2 GND, J3 +3V3, J4 GND, J5 +3V3, J6 GND, J7 Conn_01x05_Shielded, SW1 SW_SPDT, U1 LTC4054ES5-4.2, U2 LD39200D

Commit message: BreadBatt Revision 1
Parts:
- removed J5: +3V3, TestPoint:TestPoint_THTPad_2.0x2.0mm_Drill1.0mm
- removed J6: GND, TestPoint:TestPoint_THTPad_D2.0mm_Drill1.0mm
- J1: value +5Vin -> Conn_01x02; footprint TestPoint:TestPoint_THTPad_2.0x2.0mm_Drill1.0mm -> Connector_PinHeader_2.54mm:PinHeader_1x02_P2.54mm_Vertical; moved to B.Cu
- J2, J4: value GND -> Conn_01x02; footprint TestPoint:TestPoint_THTPad_D2.0mm_Drill1.0mm -> Connector_PinHeader_2.54mm:PinHeader_1x02_P2.54mm_Vertical; moved to B.Cu
- J3: value +3V3 -> Conn_01x02; footprint TestPoint:TestPoint_THTPad_2.0x2.0mm_Drill1.0mm -> Connector_PinHeader_2.54mm:PinHeader_1x02_P2.54mm_Vertical; moved to B.Cu
- moved J2 53.0 mm to (113.0, 100.3), turned to 270 degrees
- moved J3 15.2 mm to (166.4, 115.6), turned to 90 degrees
- moved J1 2.54 mm to (166.4, 100.3), turned to 90 degrees
- moved J7 2.54 mm to (168.8, 108.0)
- moved R1 1.27 mm to (140.5, 115.0)
- moved R5 0.97 mm to (148.1, 116.8)
- moved REF** 0.76 mm to (137.2, 100.8)
- moved REF** 0.76 mm to (127.0, 100.8)
- moved D2 0.51 mm to (157.5, 102.1)
- moved G*** 0.38 mm to (137.2, 106.9)
- moved C3 0.25 mm to (149.1, 113.9)
- moved C1 0.25 mm to (140.2, 112.3)
- moved C4 0.25 mm to (149.4, 112.3)
- moved R4 0.25 mm to (149.1, 115.6)
- moved U2 0.25 mm to (144.8, 113.5)
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Connections:
- J1 pad 1: +5V -> +3V3
Routing:
- net VBUS: track 8.10 -> 15.8 mm
- net Net-(C2-Pad2): track 11.0 -> 17.4 mm
- net +3V3: track 84.8 -> 83.8 mm
- net +BATT: track 67.8 -> 68.5 mm
- net Net-(C3-Pad2): track 5.40 -> 4.74 mm
- net Net-(R1-Pad2): track 34.0 -> 34.7 mm
- net -BATT: vias 0 -> 1
Other:
- board size 58.4 x 20.3 mm -> 61 x 20.3 mm
- board text added: "+"
- board text added: "+3V3"
- board text added: "+5VUSB"
- board text added: "+5Vin"
- board text added: "-"
- board text added: "BreadBatt Black (Rev. 1)"
- board text added: "GND"
- board text removed: "BreadBatt"
